File: nixieLogicV2/nixieLogicV2.kicad_pcb (KiCad board)
At the start: 2 copper layers, 138.9 x 81.3 mm, 41 parts, among them J1 GPS, J2 Conn_01x10_Female, J3 Barrel_Jack, Q1 2sk3234, SW1 SW_Push, SW2 SW_Push, SW3 SW, SW4 SW, SW5 SW, SW6 SW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

Commit message: add FirmWare Currently Ntp Function working need to add config menu
Parts:
- added R1: 10k, Resistor_SMD:R_0805_2012Metric_Pad1.15x1.40mm_HandSolder, F.Cu at (148.1, 74.9)
- added U3: 24LC64, Package_DIP:DIP-8_W7.62mm_Socket_LongPads, F.Cu at (135.9, 71.4)
- moved G*** 30.4 mm to (99.1, 118.9)
Connections:
- J3 pad 3: (no net) -> GND
- U1 pad 24: Net-(U1-Pad24) -> /WP
- U1 pad 25: Net-(U1-Pad25) -> /SW_P
- U1 pad 26: Net-(U1-Pad26) -> /1PPS
- U1 pad 33: /SW_P -> /SDA
- U1 pad 36: /1PPS -> /SCL
Routing:
- net /WP: track 0.00 -> 90.9 mm
- net /SCL: track 0.00 -> 63.8 mm
- net /SDA: track 0.00 -> 57.3 mm
- net /1PPS: track 8.49 -> 30.3 mm
- net +3V3: track 156.0 -> 174.9 mm
- net /SW_P: track 113.5 -> 105.1 mm
- net /DCDC_Vol: track 89.5 -> 92.5 mm
- net GND: track 86.1 -> 83.9 mm, vias 8 -> 14
- net Net-(D1-Pad2): track 21.4 -> 20.4 mm
Other:
- board text added: "JLCJLCJLCJLC"
